File: hardware/kicad/NOP100.kicad_pcb (KiCad board)
At the start: 4 copper layers, 100 x 85 mm, 61 parts, among them CON1 CLICK MODULE 0, CON2 CLICK MODULE 1, J1 CAN, J10 Conn_01x03, J2 Conn_01x03, J3 Conn_01x03, J4 Conn_01x03, J5 Conn_01x03, J6 Conn_01x03, J7 Conn_02x05_Odd_Even, J8 Conn_01x03, J9 Conn_01x03, Q1 BSS138, Q2 BSS138, SW1 BUS, SW2 SW_Push, U1 MURATA_MEJ2*, U2 MCP2551-I-P, U3 Teensy_4.0, U4 74HC165, U6 NCS1S1203SC

Commit message: Tweaks galore
Parts:
- removed D2: LED, Resistor_SMD:R_0805_2012Metric
- removed J7: Conn_02x05_Odd_Even, Connector_PinSocket_2.54mm:PinSocket_2x05_P2.54mm_Vertical
- removed R8: 560R, Resistor_SMD:R_0805_2012Metric
- removed the REF** at (46.0, -35.5)
- removed the REF** at (-46.0, -35.5)
- removed the REF** at (-46.0, 35.5)
- removed the REF** at (46.0, 35.5)
- added R22: 4K7 0.125W, Resistor_SMD:R_0805_2012Metric, F.Cu at (43.1, 26.0)
- added REF**: MountingHole_3.2mm_M3, MountingHole:MountingHole_3.2mm_M3, F.Cu at (-46.0, -35.5)
- added REF**: MountingHole_3.2mm_M3, MountingHole:MountingHole_3.2mm_M3, F.Cu at (-46.0, 35.5)
- added REF**: MountingHole_3.2mm_M3, MountingHole:MountingHole_3.2mm_M3, F.Cu at (46.0, -35.5)
- added REF**: MountingHole_3.2mm_M3, MountingHole:MountingHole_3.2mm_M3, F.Cu at (46.0, 35.5)
- D1: footprint LED_SMD:LED_Kingbright_APHBM2012_2x1.25mm -> Resistor_SMD:R_0805_2012Metric
- JP1: footprint Jumper:SolderJumper-2_P1.3mm_Bridged_RoundedPad1.0x1.5mm -> Jumper:SolderJumper-2_P1.3mm_Bridged_Pad1.0x1.5mm
- U3: footprint Package_DIP:DIP-28_W15.24mm -> Package_DIP:DIP-28_W15.24mm_Socket
- moved R17 12.5 mm to (45.9, -27.5)
- moved C3 5.91 mm to (-16.5, -34.3), turned to -90 degrees
- moved SW2 5.82 mm to (45.9, -23.2)
- moved D1 0.47 mm to (-46.0, -30.1), turned to 0 degrees
- turned R18 to 90 degrees
Connections:
- J10 pad 1: /OW_GND -> +3V3
- J10 pad 2: /OW_VCC -> GND
- J10 pad 3: /OW7 -> /ONEWIRE
- J2 pad 1: /OW_GND -> +3V3
- J2 pad 2: /OW_VCC -> GND
- J2 pad 3: /OW2 -> /ONEWIRE
- J3 pad 1: /OW_GND -> +3V3
- J3 pad 2: /OW_VCC -> GND
- J3 pad 3: /OW0 -> /ONEWIRE
- J4 pad 1: /OW_GND -> +3V3
- J4 pad 2: /OW_VCC -> GND
- J4 pad 3: /OW4 -> /ONEWIRE
- J5 pad 1: /OW_GND -> +3V3
- J5 pad 2: /OW_VCC -> GND
- J5 pad 3: /OW6 -> /ONEWIRE
- J6 pad 1: /OW_GND -> +3V3
- J6 pad 2: /OW_VCC -> GND
- J6 pad 3: /OW1 -> /ONEWIRE
- J8 pad 1: /OW_GND -> +3V3
- J8 pad 2: /OW_VCC -> GND
- J8 pad 3: /OW3 -> /ONEWIRE
- J9 pad 1: /OW_GND -> +3V3
- J9 pad 2: /OW_VCC -> GND
- J9 pad 3: /OW5 -> /ONEWIRE
- R18 pad 1: /SDA -> +3V3
- R18 pad 2: +3V3 -> /SDA
- U3 pad 19: /PRG_LED -> /ONEWIRE
Routing:
- net /ONEWIRE: track 0.00 -> 146.8 mm, vias 0 -> 2
- net /OW_VCC: track 92.9 -> 0.00 mm
- net /OW_GND: track 92.8 -> 0.00 mm
- net /OW1: track 72.6 -> 0.00 mm
- net /OW3: track 68.8 -> 0.00 mm
- net /OW0: track 64.8 -> 0.00 mm
- net /OW5: track 64.0 -> 0.00 mm
- net /OW7: track 59.3 -> 0.00 mm
- net /OW2: track 51.0 -> 0.00 mm
- net /OW4: track 37.2 -> 0.00 mm
- net /PRG_LED: track 28.0 -> 0.00 mm
- net +5V: track 40.7 -> 17.4 mm, vias 3 -> 2
- net GND: track 34.4 -> 13.1 mm, vias 18 -> 2
- net /OW6: track 21.0 -> 0.00 mm
- net +3V3: track 46.6 -> 49.2 mm, vias 9 -> 12
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- added copper zone on In1.Cu, net +3V3
- removed copper zone on In2.Cu, net +3V3
- removed copper zone on In1.Cu, net GND
Other:
- board text added: "TERM"
- board text removed: "0"
- board text removed: "1"
- board text removed: "2"
- board text removed: "3"
- board text removed: "4"
- board text removed: "5"
- board text removed: "6"
- board text removed: "7"
- board text removed: "INSTANCE"

Commit message: Tweaks
Parts:
- added JP2: Jumper_3_Bridged12, Connector_PinHeader_1.27mm:PinHeader_1x03_P1.27mm_Vertical, F.Cu at (35.9, 26.2)
- added JP3: Jumper_2_Open, Connector_PinHeader_1.27mm:PinHeader_1x02_P1.27mm_Vertical, F.Cu at (43.8, 26.2)
- added R8: 4K7 0.125W, Resistor_SMD:R_0805_2012Metric, F.Cu at (44.2, 29.6)
- moved R22 3.76 mm to (42.0, 29.6), turned to -90 degrees
Connections:
- J10 pad 1: +3V3 -> Net-(J10-Pin_1)
- J2 pad 1: +3V3 -> Net-(J10-Pin_1)
- J3 pad 1: +3V3 -> Net-(J10-Pin_1)
- J4 pad 1: +3V3 -> Net-(J10-Pin_1)
- J5 pad 1: +3V3 -> Net-(J10-Pin_1)
- J6 pad 1: +3V3 -> Net-(J10-Pin_1)
- J8 pad 1: +3V3 -> Net-(J10-Pin_1)
- J9 pad 1: +3V3 -> Net-(J10-Pin_1)
Routing:
- net Net-(J10-Pin_1): track 0.00 -> 85.4 mm
- net /ONEWIRE: track 146.8 -> 142.4 mm
- net Net-(JP3-A): track 0.00 -> 2.70 mm
- net +3V3: track 49.2 -> 50.0 mm, vias 12 -> 11
Other:
- board text added: "2026 (c) PDJR https://www.github.com/pdjr-n2k/NOP100"
- board text added: "NOP100 260527"
- board text added: "SW1L: ON = enable NMEA bus terminator SW1R: ON = connect NMEA shield to GND JP1: 1-Wire supply voltage (top = 5V, bot = 3.3V) JP2: 1-Wire pull-up (open = 4K7, closed = 2K35)"
- board text removed: "2024 (c) PDJR https://www.github.com/pdjr-n2k/NOP100"
- board text removed: "NOP100 2.0"
- board text removed: "PRG"
- board text removed: "TERM"
