File: hardware/kicad/NOP100.kicad_sch (KiCad schematic)
At the start: 54 parts, among them CON1 CLICK MODULE 0, CON2 CLICK MODULE 1, J1 CAN, J10 Conn_01x03, J2 Conn_01x03, J3 Conn_01x03, J4 Conn_01x03, J5 Conn_01x03, J6 Conn_01x03, J7 Conn_02x05_Odd_Even, J8 Conn_01x03, J9 Conn_01x03, Q1 BSS138, Q2 BSS138, SW1 BUS, SW2 SW_Push, U1 MURATA_MEJ2*, U2 MCP2551-I-P, U3 Teensy_4.0, U4 74HC165, U6 NCS1S1203SC

Commit message: Tweaks galore
Parts:
- removed D2: LED, Resistor_SMD:R_0805_2012Metric, symbol Device:LED
- removed J7: Conn_02x05_Odd_Even, Connector_PinSocket_2.54mm:PinSocket_2x05_P2.54mm_Vertical, symbol Connector_Generic:Conn_02x05_Odd_Even
- removed R8: 560R, Resistor_SMD:R_0805_2012Metric, symbol Device:R
- added R22: 4K7 0.125W, Resistor_SMD:R_0805_2012Metric, symbol Device:R
- D1: footprint LED_SMD:LED_Kingbright_APHBM2012_2x1.25mm -> Resistor_SMD:R_0805_2012Metric
- JP1: footprint Jumper:SolderJumper-2_P1.3mm_Bridged_RoundedPad1.0x1.5mm -> Jumper:SolderJumper-2_P1.3mm_Bridged_Pad1.0x1.5mm
- U3: footprint Package_DIP:DIP-28_W15.24mm -> Package_DIP:DIP-28_W15.24mm_Socket
Connections:
- net OW1 is gone; now on net ONEWIRE: J6.3 (Pin_3)
- net OW2 is gone; now on net ONEWIRE: J2.3 (Pin_3)
- net OW4 is gone; now on net ONEWIRE: J4.3 (Pin_3)
- net OW5 is gone; now on net ONEWIRE: J9.3 (Pin_3)
- net OW6 is gone; now on net ONEWIRE: J5.3 (Pin_3)
- net OW7 is gone; now on net ONEWIRE: J10.3 (Pin_3)
- net OW_GND is gone; now on net +3V3: J10.1 (Pin_1), J2.1 (Pin_1), J3.1 (Pin_1), J4.1 (Pin_1), J5.1 (Pin_1), J6.1 (Pin_1), J8.1 (Pin_1), J9.1 (Pin_1)
- net OW_VCC is gone; now on net GND: J10.2 (Pin_2), J2.2 (Pin_2), J3.2 (Pin_2), J4.2 (Pin_2), J5.2 (Pin_2), J6.2 (Pin_2), J8.2 (Pin_2), J9.2 (Pin_2)
- net PRG_LED is gone; now on net ONEWIRE: U3.19 (D17)
- net +3V3: now also R18.1, R22.1; no longer R18.2
- net OW3: no longer J8.3 (Pin_3)
- net SDA: now also R18.2; no longer R18.1
- net OW0 renamed ONEWIRE
- net ONEWIRE: now also J8.3 (Pin_3), R22.2
- no-connect marks 8 -> 5
Other:
- moved on the sheet: J10, J2, J3, J4, J5, J6, J8, J9, JP1, R18, R19

Commit message: Tweaks
Parts:
- added JP2: Jumper_3_Bridged12, Connector_PinHeader_1.27mm:PinHeader_1x03_P1.27mm_Vertical, symbol Jumper:Jumper_3_Bridged12
- added JP3: Jumper_2_Open, Connector_PinHeader_1.27mm:PinHeader_1x02_P1.27mm_Vertical, symbol Jumper:Jumper_2_Open
- added R8: 4K7 0.125W, Resistor_SMD:R_0805_2012Metric, symbol Device:R
Connections:
- net +3V3: now also JP2.1 (A), JP3.2 (B); no longer J10.1 (Pin_1), J2.1 (Pin_1), J3.1 (Pin_1), J4.1 (Pin_1), J5.1 (Pin_1), J6.1 (Pin_1), J8.1 (Pin_1), J9.1 (Pin_1)
- net +5V: now also JP2.3 (B)
- net ONEWIRE: now also R8.1
- new net: J10.1 (Pin_1), J2.1 (Pin_1), J3.1 (Pin_1), J4.1 (Pin_1), J5.1 (Pin_1), J6.1 (Pin_1), J8.1 (Pin_1), J9.1 (Pin_1), JP2.2 (C)
- new net: JP3.1 (A), R8.2
Other:
- title: NOP100 N2K Module with MikroBus -> NOP100 N2K Module with MikroBUS and 1-Wire
- moved on the sheet: C3, J10, J2, J3, J4, J5, J6, J8, J9, JP1, R18, R19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
